File: poe-injector/poe-injector.sch (KiCad schematic (older format))
At the start: 41 parts, among them IC1 ATTINY44-SS, J1 AVRISP6, J2 RJCSE538001, J3 RJCSE538001, Q1 SQ2361EES, Q2 2N7002K, Q3 SQ2361EES, Q4 2N7002K, U2 LTC6101, U4 LTC6101

Commit message: No, really, really bad at git merging.
Connections:
- wire segments 91 -> 71
Changed lines of the file:
@@
-EESchema Schematic File Version 2  date 8/5/2013 4:02:56 PM
+EESchema Schematic File Version 2  date 8/5/2013 4:26:51 PM
 LIBS:power
 LIBS:device
@@
 $EndDescr
 Wire Wire Line
-	4200 4050 4200 2550
-Wire Wire Line
-	4200 4050 3600 4050
+	4350 4350 3600 4350
+Wire Wire Line
+	4350 4350 4350 3300
+Wire Wire Line
+	7750 3600 7750 4450
+Wire Wire Line
+	6800 3600 5700 3600
+Wire Wire Line
+	6250 2750 6250 3300
+Wire Wire Line
+	6250 3300 4350 3300
+Wire Wire Line
+	7050 4100 7050 4400
+Wire Wire Line
+	3600 3550 4200 3550
+Wire Wire Line
+	4200 3550 4200 2550
 Wire Wire Line
 	8600 3550 8600 3450
 Wire Wire Line
-	8600 3450 4400 3450
-Wire Wire Line
-	4400 3450 4400 3550
-Wire Wire Line
-	4400 3550 3600 3550
-Wire Wire Line
 	8100 1500 8100 950
 Wire Wire Line
 	8100 950  3800 950
-Wire Wire Line
-	3800 950  3800 3450
-Wire Wire Line
-	3800 3450 3600 3450
 Connection ~ 8800 1900
 Wire Wire Line
@@
 Connection ~ 8600 2400
 Connection ~ 4700 2750
-Wire Wire Line
-	6100 3050 6250 3050
-Wire Wire Line
-	6250 2050 6400 2050
-Wire Wire Line
-	6250 2050 6250 2150
-Wire Wire Line
-	6250 2150 6150 2150
-Wire Wire Line
-	6400 2050 6400 2150
-Wire Wire Line
-	4400 2550 4350 2550
-Wire Wire Line
-	4350 2550 4350 4050
-Wire Wire Line
-	6600 5100 6900 5100
-Wire Wire Line
-	6950 4400 7050 4400
-Wire Wire Line
-	6600 4550 6600 4700
 Connection ~ 6100 2250
 Wire Wire Line
@@
 Wire Wire Line
 	5600 4200 5600 5100
-Wire Wire Line
-	5400 4200 5400 5100
-Wire Wire Line
-	8450 5050 8450 5850
-Wire Wire Line
-	8450 5850 3950 5850
-Wire Wire Line
-	3950 5850 3950 3650
-Wire Wire Line
-	3950 3650 3600 3650
 Wire Wire Line
 	3600 4450 4000 4450
@@
 	4900 4550 4900 4700
 Connection ~ 4400 2250
-Wire Wire Line
-	4400 2250 4400 2400
 Connection ~ 4900 1900
 Wire Wire Line
@@
 Wire Wire Line
 	8100 3750 8600 3750
-Wire Wire Line
-	3600 3550 4450 3550
-Wire Wire Line
-	4450 3550 4450 4050
-Wire Wire Line
-	4450 4050 4650 4050
-Wire Wire Line
-	3600 3350 3950 3350
-Wire Wire Line
-	3950 3350 3950 3250
-Wire Wire Line
-	3950 3250 4200 3250
 Wire Wire Line
 	5500 3600 5200 3600
@@
 Connection ~ 7050 4100
 Wire Wire Line
-	4100 3300 6250 3300
-Wire Wire Line
-	6250 3300 6250 2750
-Wire Wire Line
 	9750 4450 9100 4450
 Wire Wire Line
-	5900 7550 5900 7250
-Wire Wire Line
-	6400 2050 6400 1750
+	6400 1750 6400 2150
 Wire Wire Line
 	8600 2400 9600 2400
-Wire Wire Line
-	7750 3600 7750 4650
 Wire Wire Line
 	9000 3600 8350 3600
@@
 Connection ~ 1000 2450
 Wire Wire Line
-	8700 4100 8700 4650
-Wire Wire Line
 	5900 7550 5900 7250
 Connection ~ 5800 3600
@@
 	3600 4800 3600 4550
 Wire Wire Line
-	3600 3950 3850 3950
-Wire Wire Line
 	1000 3750 1000 2450
 Wire Wire Line
@@
 	6600 4550 6600 4700
 Wire Wire Line
-	7800 2700 7800 3450
-Wire Wire Line
-	7800 3450 3600 3450
-Wire Wire Line
 	5400 4200 5400 5100
 Wire Wire Line
@@
 Connection ~ 4700 2750
 Wire Wire Line
-	6450 1750 6450 1650
-Wire Wire Line
-	6450 1750 6500 1750
-Wire Wire Line
 	5400 1900 5400 2750
 Wire Wire Line
@@
 	7900 1900 8100 1900
 Wire Wire Line
-	7000 3600 7750 3600
-Wire Wire Line
-	7750 3600 7750 4450
+	7750 3600 7000 3600
 Wire Wire Line
 	7750 4450 8600 4450
 Wire Wire Line
-	3600 3650 4450 3650
-Wire Wire Line
-	4450 3650 4450 4050
+	3800 950  3800 3450
+Wire Wire Line
+	3800 3450 3600 3450
+Wire Wire Line
+	7000 4000 7000 4100
+Wire Wire Line
+	7000 4100 7150 4100
+Wire Wire Line
+	6500 1750 6350 1750
+Wire Wire Line
+	6350 1750 6350 1650
+Connection ~ 6400 1750
+Wire Wire Line
+	4650 3550 5700 3550
+Wire Wire Line
+	5700 3550 5700 3600
+Wire Wire Line
+	3600 3650 4300 3650
+Wire Wire Line
+	4300 3650 4300 3450
+Wire Wire Line
+	4300 3450 8600 3450
+Wire Wire Line
+	4450 4050 4450 3850
+Wire Wire Line
+	4450 3850 3600 3850
 $Comp
 L R R6

Commit message: Re-layout board, again
Parts:
- added R17, R18: 220k, symbol R
Connections:
- wire segments 71 -> 83

Commit message: Add resistors to drive LEDs on both ethernet jacks
Parts:
- added C2: C, symbol C
- added R19, R20, R21, R22: 330-600, symbol R
Connections:
- net +5V: now also C2.1
- net GND: now also C2.2; no longer IC1.2 ((PCINT8/CLKI/XTAL1)PB0), J2.10 (LED1+), J2.12 (LED2+), J3.10 (LED1+), J3.12 (LED2+)
- net at IC1.3 ((PCINT9/XTAL2)PB1), Q2.1 (G): now also R19.2
- net at IC1.5 ((PCINT10/CKOUT/OC0A/INT0)PB2), Q4.1 (G): now also R20.2
- new net: IC1.2 ((PCINT8/CLKI/XTAL1)PB0), R21.2, R22.1
- new net: J2.10 (LED1+), R19.1
- new net: J2.12 (LED2+), R21.1
- new net: J3.10 (LED1+), R20.1
- new net: J3.12 (LED2+), R22.2
Changed lines of the file:
@@
-EESchema Schematic File Version 2  date 8/5/2013 7:15:45 PM
+EESchema Schematic File Version 2  date 8/5/2013 8:38:49 PM
 LIBS:power
 LIBS:device
@@
 Sheet 1 1
 Title ""
-Date "5 aug 2013"
+Date "6 aug 2013"
 Rev ""
 Comp ""
@@
 $EndDescr
 Wire Wire Line
+	3600 4250 4400 4250
+Wire Wire Line
+	4400 4250 4400 3050
+Connection ~ 4200 4250
+Wire Wire Line
+	4200 4250 4200 4850
+Connection ~ 4900 4850
+Connection ~ 2050 1050
+Connection ~ 2050 1450
+Wire Wire Line
+	2350 1450 2050 1450
+Connection ~ 6900 5350
+Wire Wire Line
+	6600 5350 6900 5350
+Wire Wire Line
 	7350 4500 7350 4400
 Wire Wire Line
@@
 Connection ~ 8100 1700
 Connection ~ 6400 2050
-Connection ~ 6600 4850
 Connection ~ 8100 2400
 Connection ~ 7900 1900
@@
 	4300 3650 3600 3650
 Wire Wire Line
-	5700 3550 5700 3600
-Wire Wire Line
-	5700 3550 4650 3550
+	5700 3600 5700 3550
 Connection ~ 6400 1750
 Wire Wire Line
@@
 	7350 4100 7350 4000
 Connection ~ 7150 4100
+Wire Wire Line
+	6100 3050 6250 3050
+Connection ~ 6250 3050
+Wire Wire Line
+	2050 1050 2350 1050
+Connection ~ 4650 3550
+Connection ~ 4400 2550
+Connection ~ 3600 3950
+Wire Wire Line
+	5700 3550 4650 3550
+Wire Wire Line
+	4200 4850 4400 4850
+$Comp
+L R R21
+U 1 1 52004576
+P 4400 2800
+F 0 "R21" V 4480 2800 50  0000 C CNN
+F 1 "330-600" V 4400 2800 50  0000 C CNN
+	1    4400 2800
+	1    0    0    -1
+$EndComp
+$Comp
+L R R22
+U 1 1 5200456D
+P 4650 4850
+F 0 "R22" V 4730 4850 50  0000 C CNN
+F 1 "330-600" V 4650 4850 50  0000 C CNN
+	1    4650 4850
+	0    -1   -1   0
+$EndComp
+$Comp
+L C C2
+U 1 1 52003BA9
+P 2350 1250
+F 0 "C2" H 2400 1350 50  0000 L CNN
+F 1 "C" H 2400 1150 50  0000 L CNN
+	1    2350 1250
+	1    0    0    -1
+$EndComp
+$Comp
+L R R20
+U 1 1 52003B50
+P 6600 5100
+F 0 "R20" V 6680 5100 50  0000 C CNN
+F 1 "330-600" V 6600 5100 50  0000 C CNN
+	1    6600 5100
+	1    0    0    -1
+$EndComp
+$Comp
+L R R19
+U 1 1 52003B44
+P 6100 2800
+F 0 "R19" V 6180 2800 50  0000 C CNN
+F 1 "330-600" V 6100 2800 50  0000 C CNN
+	1    6100 2800
+	1    0    0    -1
+$EndComp
 $Comp
 L R R18
@@
 $EndComp
 $Comp
-L GND #PWR01
+L GND #PWR25
 U 1 1 52001EF2
 P 8600 3750
-F 0 "#PWR01" H 8600 3750 30  0001 C CNN
+F 0 "#PWR25" H 8600 3750 30  0001 C CNN
 F 1 "GND" H 8600 3680 30  0001 C CNN
 	1    8600 3750
@@
 $EndComp
 $Comp
-L GND #PWR02
+L GND #PWR23
 U 1 1 52001EEC
 P 8100 1700
-F 0 "#PWR02" H 8100 1700 30  0001 C CNN
+F 0 "#PWR23" H 8100 1700 30  0001 C CNN
 F 1 "GND" H 8100 1630 30  0001 C CNN
 	1    8100 1700
-	1    0    0    -1
-$EndComp
-$Comp
-L GND #PWR03
-U 1 1 52001E72
-P 3600 4250
-F 0 "#PWR03" H 3600 4250 30  0001 C CNN
-F 1 "GND" H 3600 4180 30  0001 C CNN
-	1    3600 4250
-	1    0    0    -1
-$EndComp
-$Comp
-L GND #PWR04
-U 1 1 52000F04
-P 6100 2550
-F 0 "#PWR04" H 6100 2550 30  0001 C CNN
-F 1 "GND" H 6100 2480 30  0001 C CNN
-	1    6100 2550
-	1    0    0    -1
-$EndComp
-$Comp
-L GND #PWR05
-U 1 1 52000F02
-P 4400 2550
-F 0 "#PWR05" H 4400 2550 30  0001 C CNN
-F 1 "GND" H 4400 2480 30  0001 C CNN
-	1    4400 2550
-	1    0    0    -1
-$EndComp
-$Comp
-L GND #PWR06
-U 1 1 52000EFD
-P 4900 4850
-F 0 "#PWR06" H 4900 4850 30  0001 C CNN
-F 1 "GND" H 4900 4780 30  0001 C CNN
-	1    4900 4850
-	1    0    0    -1
-$EndComp
-$Comp
-L GND #PWR07
-U 1 1 52000EFC
-P 6600 4850
-F 0 "#PWR07" H 6600 4850 30  0001 C CNN
-F 1 "GND" H 6600 4780 30  0001 C CNN
-	1    6600 4850
 	1    0    0    -1
 $EndComp
@@
 $EndComp
 $Comp
-L GND #PWR08
+L GND #PWR21
 U 1 1 5200007C
 P 7200 5100
-F 0 "#PWR08" H 7200 5100 30  0001 C CNN
+F 0 "#PWR21" H 7200 5100 30  0001 C CNN
 F 1 "GND" H 7200 5030 30  0001 C CNN
 	1    7200 5100
@@
 $EndComp
 $Comp
-L GND #PWR09
+L GND #PWR19
 U 1 1 52000076
 P 6550 2750
-F 0 "#PWR09" H 6550 2750 30  0001 C CNN
+F 0 "#PWR19" H 6550 2750 30  0001 C CNN
 F 1 "GND" H 6550 2680 30  0001 C CNN
 	1    6550 2750
@@
 $EndComp
 $Comp
-L GND #PWR010
+L GND #PWR15
 U 1 1 5113FFBF
 P 5200 3600
-F 0 "#PWR010" H 5200 3600 30  0001 C CNN
+F 0 "#PWR15" H 5200 3600 30  0001 C CNN
 F 1 "GND" H 5200 3530 30  0001 C CNN
 	1    5200 3600
@@
 $EndComp
 $Comp
-L GND #PWR011
+L GND #PWR13
 U 1 1 5113FF77
 P 4900 4550
-F 0 "#PWR011" H 4900 4550 30  0001 C CNN
+F 0 "#PWR13" H 4900 4550 30  0001 C CNN
 F 1 "GND" H 4900 4480 30  0001 C CNN
 	1    4900 4550
@@
 $EndComp
 $Comp
-L GND #PWR012
+L GND #PWR20
 U 1 1 5113FF73
 P 6600 4550
-F 0 "#PWR012" H 6600 4550 30  0001 C CNN
+F 0 "#PWR20" H 6600 4550 30  0001 C CNN
 F 1 "GND" H 6600 4480 30  0001 C CNN
 	1    6600 4550
@@
 $EndComp
 $Comp
-L GND #PWR013
+L GND #PWR9
 U 1 1 5113FD89
 P 4400 2250
-F 0 "#PWR013" H 4400 2250 30  0001 C CNN
+F 0 "#PWR9" H 4400 2250 30  0001 C CNN
 F 1 "GND" H 4400 2180 30  0001 C CNN
 	1    4400 2250
@@
 $EndComp
 $Comp
-L GND #PWR014
+L GND #PWR18
 U 1 1 5113FD86
 P 6100 2250
-F 0 "#PWR014" H 6100 2250 30  0001 C CNN
+F 0 "#PWR18" H 6100 2250 30  0001 C CNN
 F 1 "GND" H 6100 2180 30  0001 C CNN
 	1    6100 2250
@@
 $EndComp
 $Comp
-L GND #PWR015
+L GND #PWR10
 U 1 1 5113FD4C
 P 4550 2750
-F 0 "#PWR015" H 4550 2750 30  0001 C CNN
+F 0 "#PWR10" H 4550 2750 30  0001 C CNN
 F 1 "GND" H 4550 2680 30  0001 C CNN
 	1    4550 2750
@@
 $EndComp
 $Comp
-L GND #PWR016
+L GND #PWR12
 U 1 1 5113FD3D
 P 4700 1250
-F 0 "#PWR016" H 4700 1250 30  0001 C CNN
+F 0 "#PWR12" H 4700 1250 30  0001 C CNN
 F 1 "GND" H 4700 1180 30  0001 C CNN
 	1    4700 1250
@@
 $EndComp
 $Comp
-L GND #PWR017
+L GND #PWR17
 U 1 1 51132971
 P 5900 7550
-F 0 "#PWR017" H 5900 7550 30  0001 C CNN
+F 0 "#PWR17" H 5900 7550 30  0001 C CNN
 F 1 "GND" H 5900 7480 30  0001 C CNN
 	1    5900 7550
@@
 $EndComp
 $Comp
-L +5V #PWR018
+L +5V #PWR14
 U 1 1 5112C4D3
 P 5150 4050
-F 0 "#PWR018" H 5150 4140 20  0001 C CNN
+F 0 "#PWR14" H 5150 4140 20  0001 C CNN
 F 1 "+5V" H 5150 4140 30  0000 C CNN
 	1    5150 4050
@@
 $EndComp
 $Comp
-L GND #PWR019
+L GND #PWR11
 U 1 1 5112C4CE
 P 4650 4550
-F 0 "#PWR019" H 4650 4550 30  0001 C CNN
+F 0 "#PWR11" H 4650 4550 30  0001 C CNN
 F 1 "GND" H 4650 4480 30  0001 C CNN
 	1    4650 4550
@@
 $EndComp
 $Comp
-L GND #PWR020
+L GND #PWR8
 U 1 1 5112C48D
 P 4050 3050
-F 0 "#PWR020" H 4050 3050 30  0001 C CNN
+F 0 "#PWR8" H 4050 3050 30  0001 C CNN
 F 1 "GND" H 4050 2980 30  0001 C CNN
 	1    4050 3050
@@
 $EndComp
 $Comp
-L +5V #PWR021
+L +5V #PWR7
 U 1 1 5112C0CC
 P 3550 2550
-F 0 "#PWR021" H 3550 2640 20  0001 C CNN
+F 0 "#PWR7" H 3550 2640 20  0001 C CNN
 F 1 "+5V" H 3550 2640 30  0000 C CNN
 	1    3550 2550
@@
 $EndComp
 $Comp
-L +5V #PWR022
+L +5V #PWR5
 U 1 1 5111AFF4
 P 2050 1050
-F 0 "#PWR022" H 2050 1140 20  0001 C CNN
+F 0 "#PWR5" H 2050 1140 20  0001 C CNN
 F 1 "+5V" H 2050 1140 30  0000 C CNN
 	1    2050 1050
@@
 $EndComp
 $Comp
-L GND #PWR023
+L GND #PWR6
 U 1 1 5111AFED
 P 2050 1450
-F 0 "#PWR023" H 2050 1450 30  0001 C CNN
+F 0 "#PWR6" H 2050 1450 30  0001 C CNN
 F 1 "GND" H 2050 1380 30  0001 C CNN
 	1    2050 1450
@@
 $EndComp
 $Comp
-L +48V #PWR024
+L +48V #PWR27
 U 1 1 5111849B
 P 9300 3550
-F 0 "#PWR024" H 9300 3680 20  0001 C CNN
+F 0 "#PWR27" H 9300 3680 20  0001 C CNN
 F 1 "+48V" H 9300 3650 30  0000 C CNN
 	1    9300 3550
@@
 $EndComp
 $Comp
-L +48V #PWR025
+L +48V #PWR26
 U 1 1 51118493
 P 8800 1500
-F 0 "#PWR025" H 8800 1630 20  0001 C CNN
+F 0 "#PWR26" H 8800 1630 20  0001 C CNN
 F 1 "+48V" H 8800 1600 30  0000 C CNN
 	1    8800 1500
@@
 $EndComp
 $Comp
-L +48V #PWR026
+L +48V #PWR28
 U 1 1 51118467
 P 9600 2400
-F 0 "#PWR026" H 9600 2530 20  0001 C CNN
+F 0 "#PWR28" H 9600 2530 20  0001 C CNN
 F 1 "+48V" H 9600 2500 30  0000 C CNN
 	1    9600 2400
@@
 $EndComp
 $Comp
-L GND #PWR027
+L GND #PWR4
 U 1 1 51117B98
 P 1500 4550
-F 0 "#PWR027" H 1500 4550 30  0001 C CNN
+F 0 "#PWR4" H 1500 4550 30  0001 C CNN
 F 1 "GND" H 1500 4480 30  0001 C CNN
 	1    1500 4550
@@
 $EndComp
 $Comp
-L +5V #PWR028
+L +5V #PWR3
 U 1 1 51117B3E
 P 1500 3350
-F 0 "#PWR028" H 1500 3440 20  0001 C CNN
+F 0 "#PWR3" H 1500 3440 20  0001 C CNN
 F 1 "+5V" H 1500 3440 30  0000 C CNN
 	1    1500 3350
@@
 $EndComp
 $Comp
-L GND #PWR029
+L GND #PWR22
 U 1 1 5111744B
 P 7600 1500
-F 0 "#PWR029" H 7600 1500 30  0001 C CNN
+F 0 "#PWR22" H 7600 1500 30  0001 C CNN
 F 1 "GND" H 7600 1430 30  0001 C CNN
 	1    7600 1500
@@
 $EndComp
 $Comp
-L GND #PWR030
+L GND #PWR24
 U 1 1 51117447
 P 8100 3550
-F 0 "#PWR030" H 8100 3550 30  0001 C CNN
+F 0 "#PWR24" H 8100 3550 30  0001 C CNN
 F 1 "GND" H 8100 3480 30  0001 C CNN
 	1    8100 3550
@@
 $EndComp
 $Comp
-L GND #PWR031
+L GND #PWR16
 U 1 1 5110833F
 P 5200 5100
-F 0 "#PWR031" H 5200 5100 30  0001 C CNN
+F 0 "#PWR16" H 5200 5100 30  0001 C CNN
 F 1 "GND" H 5200 5030 30  0001 C CNN
 	1    5200 5100
@@
 $EndComp
 $Comp
-L +48V #PWR032
+L +48V #PWR29
 U 1 1 51106F2B
 P 9750 4450
-F 0 "#PWR032" H 9750 4580 20  0001 C CNN
+F 0 "#PWR29" H 9750 4580 20  0001 C CNN
 F 1 "+48V" H 9750 4550 30  0000 C CNN
 	1    9750 4450
@@
 $EndComp
 $Comp
-L GND #PWR033
+L GND #PWR2
 U 1 1 510E9A8D
 P 1100 1350
-F 0 "#PWR033" H 1100 1350 30  0001 C CNN
+F 0 "#PWR2" H 1100 1350 30  0001 C CNN
 F 1 "GND" H 1100 1280 30  0001 C CNN
 	1    1100 1350
@@
 $EndComp
 $Comp
-L +5V #PWR034
+L +5V #PWR1
 U 1 1 510E9A89
 P 900 1350
-F 0 "#PWR034" H 900 1440 20  0001 C CNN
+F 0 "#PWR1" H 900 1440 20  0001 C CNN
 F 1 "+5V" H 900 1440 30  0000 C CNN
 	1    900  1350
